File: pcb/esp_32_switch_board/esp_32_switch_board.kicad_pcb (KiCad board)
At the start: 2 copper layers, 109.2 x 81.3 mm, 48 parts, among them J1 Screw_Terminal_01x02, J11 Conn_01x04_Pin, J2 Screw_Terminal_01x02, J3 Screw_Terminal_01x02, J4 Screw_Terminal_01x02, J5 Screw_Terminal_01x02, J6 Conn_01x03_Pin, J7 POWER_OUT, J8 Conn_01x03_Pin, J9 Conn_01x06_Pin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

Commit message: first fully functional version
Other:
- board size 109.2 x 81.3 mm -> 114.3 x 86.4 mm
- board text added: "GND MISO CLK MOSI G25 3.3V"
- board text removed: "GND MISO CLK MOSI G5 3.3V"
